File: Eagle Files/UV_Curing_Chamber_Board/5mmtermCuringCircuit.brd (EAGLE design)
At the start: 114.8 x 100 mm, 25 parts, among them IC1 7805T, IC2 L293D, T1 RFP30N06LE, T2 RFP30N06LE

Commit message: more eagle
Parts:
- moved C1 85.5 mm to (25.4, 47.0)
- moved R1 85.5 mm to (27.9, 63.5)
- moved R2 85.5 mm to (27.9, 58.4)
- moved R3 85.5 mm to (27.9, 53.3)
- moved R5 54.3 mm to (20.3, 38.1)
Routing:
- net RELAY_NO: track 96.2 -> 0.00 mm
- net N$6: track 11.4 -> 0.00 mm
- removed copper zone on layer 16, net RELAY_NO
