File: Eagle Files/UV_Curing_Chamber_Board/5mmtermCuringCircuit.sch (EAGLE design)
At the start: 25 parts, among them IC1 7805T, IC2 L293D, T1 RFP30N06LE, T2 RFP30N06LE

Commit message: Added bypass caps to stepper outputs.
Parts:
- added C4, C5, C6, C7: 0.1u, rcl:C-US025-024X044
Connections:
- net GND: now also C4.2, C5.2, C6.2, C7.2
- net N$15: now also C4.1
- net N$23: now also C7.1
- net N$27: now also C6.1
- net N$7: now also C5.1
Changed lines of the file:
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@@
 <part name="+3V5" library="supply1" library_urn="urn:adsk.eagle:library:371" deviceset="+3V3" device=""/>
 <part name="+3V6" library="supply1" library_urn="urn:adsk.eagle:library:371" deviceset="+3V3" device=""/>
+<part name="C4" library="rcl" library_urn="urn:adsk.eagle:library:334" deviceset="C-US" device="025-024X044" package3d_urn="urn:adsk.eagle:package:23630/1" value="0.1u"/>
+<part name="C5" library="rcl" library_urn="urn:adsk.eagle:library:334" deviceset="C-US" device="025-024X044" package3d_urn="urn:adsk.eagle:package:23630/1" value="0.1u"/>
+<part name="C6" library="rcl" library_urn="urn:adsk.eagle:library:334" deviceset="C-US" device="025-024X044" package3d_urn="urn:adsk.eagle:package:23630/1" value="0.1u"/>
+<part name="C7" library="rcl" library_urn="urn:adsk.eagle:library:334" deviceset="C-US" device="025-024X044" package3d_urn="urn:adsk.eagle:package:23630/1" value="0.1u"/>
+<part name="GND6" library="supply1" library_urn="urn:adsk.eagle:library:371" deviceset="GND" device=""/>
+<part name="GND18" library="supply1" library_urn="urn:adsk.eagle:library:371" deviceset="GND" device=""/>
+<part name="GND19" library="supply1" library_urn="urn:adsk.eagle:library:371" deviceset="GND" device=""/>
+<part name="GND20" library="supply1" library_urn="urn:adsk.eagle:library:371" deviceset="GND" device=""/>
 </parts>
 <sheets>
@@
 <attribute name="VALUE" x="307.34" y="157.48" size="1.778" layer="96" rot="R90"/>
 </instance>
+<instance part="C4" gate="G$1" x="233.68" y="104.14" smashed="yes" rot="R270">
+<attribute name="NAME" x="234.315" y="103.124" size="1.778" layer="95" rot="R270"/>
+<attribute name="VALUE" x="229.489" y="103.124" size="1.778" layer="96" rot="R270"/>
+</instance>
+<instance part="C5" gate="G$1" x="233.68" y="88.9" smashed="yes" rot="R270">
+<attribute name="NAME" x="234.315" y="87.884" size="1.778" layer="95" rot="R270"/>
+<attribute name="VALUE" x="229.489" y="87.884" size="1.778" layer="96" rot="R270"/>
+</instance>
+<instance part="C6" gate="G$1" x="307.34" y="104.14" smashed="yes" rot="R90">
+<attribute name="NAME" x="306.705" y="105.156" size="1.778" layer="95" rot="R90"/>
+<attribute name="VALUE" x="311.531" y="105.156" size="1.778" layer="96" rot="R90"/>
+</instance>
+<instance part="C7" gate="G$1" x="307.34" y="88.9" smashed="yes" rot="R90">
+<attribute name="NAME" x="306.705" y="89.916" size="1.778" layer="95" rot="R90"/>
+<attribute name="VALUE" x="311.531" y="89.916" size="1.778" layer="96" rot="R90"/>
+</instance>
+<instance part="GND6" gate="1" x="314.96" y="96.52" smashed="yes">
+<attribute name="VALUE" x="312.42" y="93.98" size="1.778" layer="96"/>
+</instance>
+<instance part="GND18" gate="1" x="314.96" y="81.28" smashed="yes">
+<attribute name="VALUE" x="312.42" y="78.74" size="1.778" layer="96"/>
+</instance>
+<instance part="GND19" gate="1" x="226.06" y="99.06" smashed="yes">
+<attribute name="VALUE" x="223.52" y="96.52" size="1.778" layer="96"/>
+</instance>
+<instance part="GND20" gate="1" x="226.06" y="73.66" smashed="yes">
+<attribute name="VALUE" x="223.52" y="71.12" size="1.778" layer="96"/>
+</instance>
 </instances>
 <busses>
@@
 <pinref part="GND15" gate="1" pin="GND"/>
 <wire x1="347.98" y1="228.6" x2="353.06" y2="228.6" width="0.1524" layer="91"/>
+</segment>
+<segment>
+<pinref part="C4" gate="G$1" pin="2"/>
+<wire x1="228.6" y1="104.14" x2="226.06" y2="104.14" width="0.1524" layer="91"/>
+<pinref part="GND19" gate="1" pin="GND"/>
+<wire x1="226.06" y1="104.14" x2="226.06" y2="101.6" width="0.1524" layer="91"/>
+</segment>
+<segment>
+<pinref part="C5" gate="G$1" pin="2"/>
+<wire x1="228.6" y1="88.9" x2="226.06" y2="88.9" width="0.1524" layer="91"/>
+<pinref part="GND20" gate="1" pin="GND"/>
+<wire x1="226.06" y1="88.9" x2="226.06" y2="76.2" width="0.1524" layer="91"/>
+</segment>
+<segment>
+<pinref part="C6" gate="G$1" pin="2"/>
+<wire x1="312.42" y1="104.14" x2="314.96" y2="104.14" width="0.1524" layer="91"/>
+<pinref part="GND6" gate="1" pin="GND"/>
+<wire x1="314.96" y1="104.14" x2="314.96" y2="99.06" width="0.1524" layer="91"/>
+</segment>
+<segment>
+<pinref part="C7" gate="G$1" pin="2"/>
+<wire x1="312.42" y1="88.9" x2="314.96" y2="88.9" width="0.1524" layer="91"/>
+<pinref part="GND18" gate="1" pin="GND"/>
+<wire x1="314.96" y1="88.9" x2="314.96" y2="83.82" width="0.1524" layer="91"/>
 </segment>
 </net>
@@
 <pinref part="MOTOR_BREAKOUT" gate="1" pin="2"/>
 <wire x1="261.62" y1="71.12" x2="261.62" y2="63.5" width="0.1524" layer="91"/>
+<pinref part="C5" gate="G$1" pin="1"/>
+<wire x1="236.22" y1="88.9" x2="248.92" y2="88.9" width="0.1524" layer="91"/>
+<junction x="248.92" y="88.9"/>
 </segment>
 </net>
@@
 <pinref part="MOTOR_BREAKOUT" gate="1" pin="1"/>
 <wire x1="259.08" y1="68.58" x2="259.08" y2="63.5" width="0.1524" layer="91"/>
+<pinref part="C4" gate="G$1" pin="1"/>
+<wire x1="236.22" y1="104.14" x2="241.3" y2="104.14" width="0.1524" layer="91"/>
+<junction x="241.3" y="104.14"/>
 </segment>
 </net>
@@
 <pinref part="MOTOR_BREAKOUT" gate="1" pin="3"/>
 <wire x1="264.16" y1="71.12" x2="264.16" y2="63.5" width="0.1524" layer="91"/>
+<pinref part="C7" gate="G$1" pin="1"/>
+<wire x1="294.64" y1="88.9" x2="304.8" y2="88.9" width="0.1524" layer="91"/>
+<junction x="294.64" y="88.9"/>
 </segment>
 </net>
@@
 <pinref part="MOTOR_BREAKOUT" gate="1" pin="4"/>
 <wire x1="266.7" y1="68.58" x2="266.7" y2="63.5" width="0.1524" layer="91"/>
-</segment>
-</net>
+<pinref part="C6" gate="G$1" pin="1"/>
+<wire x1="297.18" y1="104.14" x2="304.8" y2="104.14" width="0.1524" layer="91"/>
+<junction x="297.18" y="104.14"/>
+</segment>
+</net>
