File: Eagle Files/UV_Curing_Chamber_Board/v3/newbottomboard.brd (EAGLE design)
At the start: 143.3 x 88.5 mm, 29 parts, among them IC1 7805T, IC2 L293D, T1 RFP30N06LE, T2 RFP30N06LE

Commit message: updating v3 board
Parts:
- moved ROTARY_ENC 11.6 mm to (56.2, 81.7)
Routing:
- net +3V3: track 187.9 -> 203.5 mm
- net N$19: track 42.6 -> 54.1 mm
- net N$18: track 26.0 -> 28.2 mm
Changed lines of the file:
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@@
 <attribute name="VALUE" x="82.16" y="2.54" size="0.6096" layer="27" font="vector" ratio="20" rot="R180"/>
 </element>
-<element name="ROTARY_ENC" library="SparkFun-Connectors" library_urn="urn:adsk.eagle:library:513" package="1X05" package3d_urn="urn:adsk.eagle:package:38104/1" value="" x="67.85" y="82.14" smashed="yes">
-<attribute name="NAME" x="66.58" y="83.537" size="0.6096" layer="25" font="vector" ratio="20"/>
-<attribute name="VALUE" x="66.58" y="80.108" size="0.6096" layer="27" font="vector" ratio="20"/>
+<element name="ROTARY_ENC" library="SparkFun-Connectors" library_urn="urn:adsk.eagle:library:513" package="1X05" package3d_urn="urn:adsk.eagle:package:38104/1" value="" x="56.25" y="81.74" smashed="yes">
+<attribute name="NAME" x="54.98" y="83.137" size="0.6096" layer="25" font="vector" ratio="20"/>
+<attribute name="VALUE" x="54.98" y="79.708" size="0.6096" layer="27" font="vector" ratio="20"/>
 </element>
 <element name="SPEAKER" library="SparkFun-Connectors" library_urn="urn:adsk.eagle:library:513" package="SCREWTERMINAL-5MM-2" package3d_urn="urn:adsk.eagle:package:38044/1" value="" x="115.2" y="2.89" smashed="yes">
@@
 <contactref element="ROTARY_ENC" pad="3"/>
 <contactref element="U$1" pad="5"/>
-<wire x1="73.025" y1="74.93" x2="73.025" y2="81.915" width="0.508" layer="16"/>
-<wire x1="71.12" y1="73.025" x2="73.025" y2="74.93" width="0.508" layer="16"/>
-<wire x1="71.12" y1="60.96" x2="71.12" y2="73.025" width="0.508" layer="16"/>
-<wire x1="68.58" y1="58.42" x2="71.12" y2="60.96" width="0.508" layer="16"/>
-<wire x1="73.025" y1="81.915" x2="72.93" y2="82.14" width="0.508" layer="16"/>
-<wire x1="68.58" y1="58.42" x2="68.2" y2="58.43" width="0.508" layer="16"/>
+<wire x1="68.2" y1="58.43" x2="68.2" y2="58.706975" width="0.508" layer="16"/>
+<wire x1="67.6154" y1="75.4546" x2="61.33" y2="81.74" width="0.508" layer="16"/>
+<wire x1="68.2" y1="58.706975" x2="69.8002" y2="60.307175" width="0.508" layer="16"/>
+<wire x1="68.77553125" y1="75.4546" x2="67.6154" y2="75.4546" width="0.508" layer="16"/>
+<wire x1="69.8002" y1="60.307175" x2="69.8002" y2="74.42993125" width="0.508" layer="16"/>
+<wire x1="69.8002" y1="74.42993125" x2="68.77553125" y2="75.4546" width="0.508" layer="16"/>
 </signal>
 <signal name="N$19">
 <contactref element="ROTARY_ENC" pad="4"/>
 <contactref element="U$1" pad="7"/>
-<wire x1="78.105" y1="85.09" x2="75.565" y2="82.55" width="0.508" layer="16"/>
-<wire x1="78.74" y1="85.09" x2="78.105" y2="85.09" width="0.508" layer="16"/>
-<wire x1="80.645" y1="83.185" x2="78.74" y2="85.09" width="0.508" layer="16"/>
 <wire x1="80.645" y1="78.74" x2="80.645" y2="83.185" width="0.508" layer="16"/>
 <wire x1="73.66" y1="71.755" x2="80.645" y2="78.74" width="0.508" layer="16"/>
 <wire x1="73.66" y1="58.42" x2="73.66" y2="71.755" width="0.508" layer="16"/>
 <wire x1="68.58" y1="53.34" x2="73.66" y2="58.42" width="0.508" layer="16"/>
-<wire x1="75.565" y1="82.55" x2="75.47" y2="82.14" width="0.508" layer="16"/>
 <wire x1="68.58" y1="53.34" x2="68.2" y2="53.35" width="0.508" layer="16"/>
+<wire x1="80.645" y1="83.185" x2="79.78" y2="84.05" width="0.508" layer="16"/>
+<wire x1="79.78" y1="84.05" x2="64.8" y2="84.05" width="0.508" layer="16"/>
+<wire x1="64.8" y1="84.05" x2="63.87" y2="83.12" width="0.508" layer="16"/>
+<wire x1="63.87" y1="83.12" x2="63.87" y2="81.74" width="0.508" layer="16"/>
 </signal>
 <signal name="N$20">
 <contactref element="ROTARY_ENC" pad="5"/>
 <contactref element="U$1" pad="6"/>
-<wire x1="78.105" y1="78.74" x2="78.105" y2="81.915" width="0.508" layer="16"/>
-<wire x1="72.39" y1="73.025" x2="78.105" y2="78.74" width="0.508" layer="16"/>
-<wire x1="72.39" y1="59.69" x2="72.39" y2="73.025" width="0.508" layer="16"/>
 <wire x1="68.58" y1="55.88" x2="72.39" y2="59.69" width="0.508" layer="16"/>
-<wire x1="78.105" y1="81.915" x2="78.01" y2="82.14" width="0.508" layer="16"/>
 <wire x1="68.58" y1="55.88" x2="68.2" y2="55.89" width="0.508" layer="16"/>
+<wire x1="72.39" y1="75.76" x2="66.41" y2="81.74" width="0.508" layer="16"/>
+<wire x1="72.39" y1="59.69" x2="72.39" y2="75.76" width="0.508" layer="16"/>
 </signal>
 <signal name="N$17">
@@
 <wire x1="68.58" y1="69.215" x2="68.58" y2="74.295" width="0.508" layer="16"/>
 <wire x1="68.58" y1="69.215" x2="68.2" y2="68.59" width="0.508" layer="16"/>
-<wire x1="70.485" y1="76.2" x2="70.485" y2="81.915" width="0.508" layer="16"/>
-<wire x1="68.58" y1="74.295" x2="70.485" y2="76.2" width="0.508" layer="16"/>
-<wire x1="70.485" y1="81.915" x2="70.39" y2="82.14" width="0.508" layer="16"/>
 <wire x1="68.58" y1="74.295" x2="68.26" y2="74.21" width="0.508" layer="16"/>
 <wire x1="138.43" y1="77.47" x2="135.89" y2="80.01" width="0.508" layer="16"/>
@@
 <wire x1="139.7" y1="55.245" x2="139.7" y2="19.685" width="0.508" layer="16"/>
 <wire x1="137.795" y1="57.15" x2="139.7" y2="55.245" width="0.508" layer="16"/>
-<wire x1="74.295" y1="86.36" x2="70.485" y2="82.55" width="0.508" layer="16"/>
-<wire x1="129.54" y1="86.36" x2="74.295" y2="86.36" width="0.508" layer="16"/>
 <wire x1="135.89" y1="80.01" x2="129.54" y2="86.36" width="0.508" layer="16"/>
-<wire x1="70.485" y1="82.55" x2="70.39" y2="82.14" width="0.508" layer="16"/>
 <wire x1="135.89" y1="80.01" x2="135.5" y2="80.01" width="0.508" layer="16"/>
+<wire x1="68.26" y1="74.21" x2="66.32" y2="74.21" width="0.508" layer="16"/>
+<wire x1="66.32" y1="74.21" x2="58.79" y2="81.74" width="0.508" layer="16"/>
+<wire x1="63.41" y1="86.36" x2="58.79" y2="81.74" width="0.508" layer="16"/>
+<wire x1="129.54" y1="86.36" x2="63.41" y2="86.36" width="0.508" layer="16"/>
 </signal>
 <signal name="N$1">
